File: matrix_rgb.kicad_sch (KiCad schematic)
At the start: 218 parts, among them K1 ESC, K10 F9, K11 F10, K12 F11, K13 F12, K14 PRTSCR, K15 DELETE, K16 INSERT, K17 BACKTICK, K18 1, K19 2, K2 F1, K20 3, K21 4, K22 5, K23 6, K24 7, K25 8, K26 9, K27 0, K28 MINUS, K29 EQUAL, K3 F2, K30 BACKSPACE, K31 HOME, K32 TAB, K33 Q, K34 W, K35 E, K36 R, K37 T, K38 Y, K39 U, K4 F3, K40 I, K41 O, K42 P, K43 OBRAC, K44 CBRAC, K45 PAGEUP, K46 CAPS, K47 A, K48 S, K49 D, K5 F4, K50 F, K51 G, K52 H, K53 J, K54 K, K55 L, K56 SEMICOLON, K57 QUOTE, K58 HASH, K59 ISO ENTER, K6 F5, K60 PAGEDOWN, K61 LSHIFT, K62 BCKSLASH, K63 Z, K64 X, K65 C, K66 V, K67 B, K68 N, K69 M, K7 F6, K70 COMMA, K71 DOT, K72 SLASH, K73 RSHIFT, K74 UP, K75 END, K76 LCTRL, K77 LWIN, K78 LALT, K79 SPACE, K8 F7, K80 RALT(ALTGR), K81 FN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

Commit message: Matrix
Parts:
- removed LED1, LED10, LED11, LED12, LED13, LED14, LED15, LED16, LED17, LED18, LED19, LED2, LED20, LED21, LED22, LED23, LED24, LED25, LED3, LED4, LED5, LED6, LED7, LED8, LED9: HH-SMD6028RGBC-CA, marbastlib-mx:LED_MX_6028R, symbol Device:LED_GRBA
- added LED10, LED11, LED12, LED13, LED14, LED15, LED16, LED17, LED18, LED19, LED2, LED20, LED21, LED22, LED23, LED24, LED25, LED3, LED4, LED5, LED6, LED7, LED8, LED9: MHT151RGBCT, LED-RGB:MHT151RGBCT-RGB-Reverse-Mount-1206, symbol Device:LED_ABGR
- gave numbers to parts that had none: 1
Connections:
- net CS1: now also LED1.2 (BK), LED2.2 (BK), LED3.2 (BK), LED4.2 (BK), LED5.2 (BK), LED6.2 (BK), LED7.2 (BK), LED8.2 (BK), LED9.2 (BK)
- net CS19: now also LED10.2 (BK), LED11.2 (BK), LED12.2 (BK), LED13.2 (BK), LED14.4 (RK), LED15.2 (BK), LED16.2 (BK)
- net CS2: now also LED1.3 (GK), LED2.3 (GK), LED3.3 (GK), LED4.3 (GK), LED5.3 (GK), LED6.3 (GK), LED7.3 (GK), LED8.3 (GK), LED9.3 (GK)
- net CS20: now also LED10.3 (GK), LED11.3 (GK), LED12.3 (GK), LED13.3 (GK), LED14.3 (GK), LED15.3 (GK), LED16.3 (GK)
- net CS21: now also LED10.4 (RK), LED11.4 (RK), LED12.4 (RK), LED13.4 (RK), LED14.2 (BK), LED15.4 (RK), LED16.4 (RK)
- net CS3: now also LED1.4 (RK), LED2.4 (RK), LED3.4 (RK), LED4.4 (RK), LED5.4 (RK), LED6.4 (RK), LED7.4 (RK), LED8.4 (RK), LED9.4 (RK)
- net CS4: now also LED17.2 (BK), LED18.2 (BK), LED19.2 (BK), LED20.2 (BK), LED21.2 (BK), LED22.2 (BK), LED23.2 (BK), LED24.2 (BK), LED25.2 (BK)
- net CS5: now also LED17.3 (GK), LED18.3 (GK), LED19.3 (GK), LED20.3 (GK), LED21.3 (GK), LED22.3 (GK), LED23.3 (GK), LED24.3 (GK), LED25.3 (GK)
- net CS6: now also LED17.4 (RK), LED18.4 (RK), LED19.4 (RK), LED20.4 (RK), LED21.4 (RK), LED22.4 (RK), LED23.4 (RK), LED24.4 (RK), LED25.4 (RK)
- net SW1: now also LED10.1 (A), LED25.1 (A), LED9.1 (A)
- net SW2: now also LED11.1 (A), LED24.1 (A), LED8.1 (A)
- net SW3: now also LED12.1 (A), LED23.1 (A), LED7.1 (A)
- net SW4: now also LED13.1 (A), LED22.1 (A), LED6.1 (A)
- net SW5: now also LED14.1 (A), LED21.1 (A), LED5.1 (A)
- net SW6: now also LED15.1 (A), LED20.1 (A), LED4.1 (A)
- net SW7: now also LED16.1 (A), LED19.1 (A), LED3.1 (A)
- net SW8: now also LED18.1 (A), LED2.1 (A)
- net SW9: now also LED1.1 (A), LED17.1 (A)
Other:
- moved on the sheet: LED1

Commit message: Matrix
Parts:
- removed LED26, LED27, LED28, LED29, LED30, LED31: HH-SMD6028RGBC-CA, marbastlib-mx:LED_MX_6028R, symbol Device:LED_GRBA
- added LED26, LED27, LED28, LED29, LED30, LED31: MHT151RGBCT, LED-RGB:MHT151RGBCT-RGB-Reverse-Mount-1206, symbol Device:LED_ABGR
Connections:
- net CS22: now also LED26.2 (BK), LED27.2 (BK), LED28.2 (BK), LED29.2 (BK), LED30.2 (BK), LED31.2 (BK)
- net CS23: now also LED26.3 (GK), LED27.3 (GK), LED28.3 (GK), LED29.3 (GK), LED30.3 (GK), LED31.3 (GK)
- net CS24: now also LED26.4 (RK), LED27.4 (RK), LED28.4 (RK), LED29.4 (RK), LED30.4 (RK), LED31.4 (RK)
- net SW1: now also LED26.1 (A)
- net SW2: now also LED27.1 (A)
- net SW3: now also LED28.1 (A)
- net SW4: now also LED29.1 (A)
- net SW6: now also LED30.1 (A)
- net SW7: now also LED31.1 (A)

Commit message: Matrix
Parts:
- removed LED32, LED33, LED34, LED35, LED36, LED37, LED38, LED39, LED40, LED41, LED42, LED43, LED44: HH-SMD6028RGBC-CA, marbastlib-mx:LED_MX_6028R, symbol Device:LED_GRBA
- added LED32, LED33, LED34, LED35, LED36, LED37, LED38, LED39, LED40, LED41, LED42, LED43, LED44: MHT151RGBCT, LED-RGB:MHT151RGBCT-RGB-Reverse-Mount-1206, symbol Device:LED_ABGR
Connections:
- net CS25: now also LED40.2 (BK), LED41.2 (BK), LED42.2 (BK), LED43.2 (BK), LED44.2 (BK)
- net CS26: now also LED40.3 (GK), LED41.3 (GK), LED42.3 (GK), LED43.3 (GK), LED44.3 (GK)
- net CS27: now also LED40.4 (RK), LED41.4 (RK), LED42.4 (RK), LED43.4 (RK), LED44.4 (RK)
- net CS7: now also LED32.2 (BK), LED33.2 (BK), LED34.2 (BK), LED35.2 (BK), LED36.2 (BK), LED37.2 (BK), LED38.2 (BK), LED39.2 (BK)
- net CS8: now also LED32.3 (GK), LED33.3 (GK), LED34.3 (GK), LED35.3 (GK), LED36.3 (GK), LED37.3 (GK), LED38.3 (GK), LED39.3 (GK)
- net CS9: now also LED32.4 (RK), LED33.4 (RK), LED34.4 (RK), LED35.4 (RK), LED36.4 (RK), LED37.4 (RK), LED38.4 (RK), LED39.4 (RK)
- net SW1: now also LED39.1 (A), LED40.1 (A)
- net SW2: now also LED38.1 (A)
- net SW3: now also LED37.1 (A), LED42.1 (A)
- net SW4: now also LED36.1 (A), LED43.1 (A)
- net SW5: now also LED35.1 (A), LED44.1 (A)
- net SW6: now also LED34.1 (A)
- net SW7: now also LED33.1 (A)
- net SW9: now also LED32.1 (A)

Commit message: Schematic
Parts:
- removed LED45, LED46, LED47, LED48, LED49, LED50, LED51: HH-SMD6028RGBC-CA, marbastlib-mx:LED_MX_6028R, symbol Device:LED_GRBA
- added LED45, LED46, LED47, LED48, LED49, LED50, LED51: MHT151RGBCT, LED-RGB:MHT151RGBCT-RGB-Reverse-Mount-1206, symbol Device:LED_ABGR
Connections:
- net CS10: now also LED46.2 (BK), LED47.2 (BK), LED48.2 (BK), LED49.2 (BK), LED50.2 (BK), LED51.2 (BK)
- net CS11: now also LED46.3 (GK), LED47.3 (GK), LED48.3 (GK), LED49.3 (GK), LED50.3 (GK), LED51.3 (GK)
- net CS12: now also LED46.4 (RK), LED47.4 (RK), LED48.4 (RK), LED49.4 (RK), LED50.4 (RK), LED51.4 (RK)
- net CS25: now also LED45.2 (BK)
- net CS26: now also LED45.3 (GK)
- net CS27: now also LED45.4 (RK)
- net SW3: now also LED51.1 (A)
- net SW4: now also LED50.1 (A)
- net SW5: now also LED49.1 (A)
- net SW6: now also LED48.1 (A)
- net SW7: now also LED45.1 (A), LED47.1 (A)
- net SW9: now also LED46.1 (A)

Commit message: Matrix Schematic
Parts:
- removed LED52, LED53, LED54, LED55, LED56, LED57, LED58, LED59, LED60: HH-SMD6028RGBC-CA, marbastlib-mx:LED_MX_6028R, symbol Device:LED_GRBA
- added LED52, LED53, LED54, LED55, LED56, LED57, LED58, LED59, LED60: MHT151RGBCT, LED-RGB:MHT151RGBCT-RGB-Reverse-Mount-1206, symbol Device:LED_ABGR
Connections:
- net CS10: now also LED52.2 (BK), LED53.2 (BK)
- net CS11: now also LED52.3 (GK), LED53.3 (GK)
- net CS12: now also LED52.4 (RK), LED53.4 (RK)
- net CS28: now also LED54.3 (GK), LED55.2 (BK), LED56.2 (BK), LED57.2 (BK), LED58.2 (BK), LED59.2 (BK), LED60.2 (BK)
- net CS29: now also LED54.4 (RK), LED55.3 (GK), LED56.3 (GK), LED57.3 (GK), LED58.3 (GK), LED59.3 (GK), LED60.3 (GK)
- net CS30: now also LED54.2 (BK), LED55.4 (RK), LED56.4 (RK), LED57.4 (RK), LED58.4 (RK), LED59.4 (RK), LED60.4 (RK)
- net SW1: now also LED53.1 (A), LED54.1 (A)
- net SW2: now also LED41.1 (A), LED52.1 (A), LED55.1 (A)
- net SW3: now also LED56.1 (A)
- net SW4: now also LED57.1 (A)
- net SW5: now also LED58.1 (A)
- net SW6: now also LED59.1 (A)
- net SW7: now also LED60.1 (A)

Commit message: Schematic
Parts:
- removed LED61, LED62, LED63, LED64, LED65, LED66, LED67, LED68, LED69, LED70, LED71, LED72, LED73, LED74, LED75, LED76, LED77, LED78, LED79, LED80, LED81, LED82, LED83, LED84: HH-SMD6028RGBC-CA, marbastlib-mx:LED_MX_6028R, symbol Device:LED_GRBA
- added LED61, LED62, LED63, LED64, LED65, LED66, LED67, LED68, LED69, LED70, LED71, LED72, LED73, LED74, LED75, LED76, LED77, LED78, LED79, LED80, LED81, LED82, LED83, LED84: MHT151RGBCT, PCM_marbastlib-xp-mx:LED_MX_1206R, symbol Device:LED_ABGR
- K1, K10, K11, K12, K13, K14, K15, K16, K17, K18, K19, K2, K20, K21, K22, K23, K24, K25, K26, K27, K28, K29, K3, K30, K31, K33, K34, K35, K36, K37, K38, K39, K4, K40, K41, K42, K43, K44, K45, K47, K48, K49, K5, K50, K51, K52, K53, K54, K55, K56, K57, K58, K59, K6, K60, K62, K63, K64, K65, K66, K67, K68, K69, K7, K70, K71, K72, K74, K75, K79, K8, K82, K83, K84, K9: footprint marbastlib-mx:SW_MX_HS_1u -> PCM_marbastlib-mx:SW_MX_HS_1u
- K32: footprint marbastlib-mx:SW_MX_HS_1.5u -> PCM_marbastlib-mx:SW_MX_HS_1.5u
- K46, K73: footprint marbastlib-mx:SW_MX_HS_1.75u -> PCM_marbastlib-mx:SW_MX_HS_1.75u
- K61, K76, K77, K78, K80, K81: footprint marbastlib-mx:SW_MX_HS_1.25u -> PCM_marbastlib-mx:SW_MX_HS_1.25u
- LED1, LED10, LED11, LED12, LED13, LED14, LED15, LED16, LED17, LED18, LED19, LED2, LED20, LED21, LED22, LED23, LED24, LED25, LED26, LED27, LED28, LED29, LED3, LED30, LED31, LED32, LED33, LED34, LED35, LED36, LED37, LED38, LED39, LED4, LED40, LED41, LED42, LED43, LED44, LED45, LED46, LED47, LED48, LED49, LED5, LED50, LED51, LED52, LED53, LED54, LED55, LED56, LED57, LED58, LED59, LED6, LED60, LED7, LED8, LED9: footprint LED-RGB:MHT151RGBCT-RGB-Reverse-Mount-1206 -> PCM_marbastlib-xp-mx:LED_MX_1206R
- S1: footprint marbastlib-mx:STAB_MX_6.25u -> PCM_marbastlib-mx:STAB_MX_6.25u
- S2: footprint marbastlib-mx:STAB_MX_2u -> PCM_marbastlib-mx:STAB_MX_2u
- S3: footprint marbastlib-mx:STAB_MX_ISO -> PCM_marbastlib-mx:STAB_MX_ISO
Connections:
- net CS13: now also LED61.2 (BK), LED62.2 (BK), LED63.2 (BK), LED64.2 (BK), LED65.2 (BK), LED66.2 (BK), LED67.2 (BK), LED68.2 (BK), LED69.2 (BK)
- net CS14: now also LED61.3 (GK), LED62.3 (GK), LED63.3 (GK), LED64.3 (GK), LED65.3 (GK), LED66.3 (GK), LED67.3 (GK), LED68.3 (GK), LED69.3 (GK)
- net CS15: now also LED61.4 (RK), LED62.4 (RK), LED63.4 (RK), LED64.4 (RK), LED65.4 (RK), LED66.4 (RK), LED67.4 (RK), LED68.4 (RK), LED69.4 (RK)
- net CS16: now also LED70.2 (BK), LED71.2 (BK), LED72.2 (BK), LED73.2 (BK), LED74.2 (BK), LED75.2 (BK)
- net CS17: now also LED70.3 (GK), LED71.3 (GK), LED72.3 (GK), LED73.3 (GK), LED74.3 (GK), LED75.3 (GK)
- net CS18: now also LED70.4 (RK), LED71.4 (RK), LED72.4 (RK), LED73.4 (RK), LED74.4 (RK), LED75.4 (RK)
- net CS31: now also LED76.2 (BK), LED77.2 (BK), LED78.2 (BK), LED79.2 (BK), LED80.2 (BK), LED81.2 (BK), LED82.2 (BK), LED83.2 (BK), LED84.2 (BK)
- net CS32: now also LED76.3 (GK), LED77.3 (GK), LED78.3 (GK), LED79.3 (GK), LED80.3 (GK), LED81.3 (GK), LED82.3 (GK), LED83.3 (GK), LED84.3 (GK)
- net CS33: now also LED76.4 (RK), LED77.4 (RK), LED78.4 (RK), LED79.4 (RK), LED80.4 (RK), LED81.4 (RK), LED82.4 (RK), LED83.4 (RK), LED84.4 (RK)
- net SW1: now also LED69.1 (A), LED70.1 (A)
- net SW2: now also LED68.1 (A), LED71.1 (A), LED80.1 (A)
- net SW3: now also LED67.1 (A), LED72.1 (A), LED79.1 (A), LED81.1 (A)
- net SW4: now also LED66.1 (A)
- net SW5: now also LED65.1 (A), LED73.1 (A), LED82.1 (A)
- net SW6: now also LED64.1 (A), LED74.1 (A), LED83.1 (A)
- net SW7: now also LED63.1 (A), LED75.1 (A), LED78.1 (A), LED84.1 (A)
- net SW8: now also LED62.1 (A), LED77.1 (A)
- net SW9: now also LED61.1 (A), LED76.1 (A)

Commit message: Matrix
Changed footprints to 1206 ROT
Parts:
- LED1, LED10, LED11, LED12, LED13, LED14, LED15, LED16, LED17, LED18, LED19, LED2, LED20, LED21, LED22, LED23, LED24, LED25, LED26, LED27, LED28, LED29, LED3, LED30, LED31, LED32, LED33, LED34, LED35, LED36, LED37, LED38, LED39, LED4, LED40, LED41, LED42, LED43, LED44, LED45, LED46, LED47, LED48, LED49, LED5, LED50, LED51, LED52, LED53, LED54, LED55, LED56, LED57, LED58, LED59, LED6, LED60, LED61, LED62, LED63, LED64, LED65, LED66, LED67, LED68, LED69, LED7, LED70, LED71, LED72, LED73, LED74, LED75, LED76, LED77, LED78, LED79, LED8, LED80, LED81, LED82, LED83, LED84, LED9: footprint PCM_marbastlib-xp-mx:LED_MX_1206R -> PCM_marbastlib-xp-mx:LED_MX_1206R-ROT

Commit message: PCB
Connections:
- net CS19: now also LED14.2 (BK); no longer LED14.4 (RK)
- net CS21: now also LED14.4 (RK); no longer LED14.2 (BK)
Changed lines of the file:
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@@
     )
   )
-  (global_label "CS21" (shape input) (at 398.272 249.174 180) (fields_autoplaced)
-    (effects (font (size 1.27 1.27)) (justify right))
-    (property "Intersheetrefs" "${INTERSHEET_REFS}" (at 390.9603 249.0946 0)
+  (global_label "CS21" (shape input) (at 398.272 239.014 180) (fields_autoplaced)
+    (effects (font (size 1.27 1.27)) (justify right))
+    (property "Intersheetrefs" "${INTERSHEET_REFS}" (at 390.9603 238.9346 0)
       (effects (font (size 1.27 1.27)) (justify right) hide)
     )
@@
     )
   )
-  (global_label "CS19" (shape input) (at 398.272 239.014 180) (fields_autoplaced)
-    (effects (font (size 1.27 1.27)) (justify right))
-    (property "Intersheetrefs" "${INTERSHEET_REFS}" (at 390.9603 238.9346 0)
-      (effects (font (size 1.27 1.27)) (justify right) hide)
-    )
+  (global_label "CS19" (shape input) (at 398.272 249.174 180) (fields_autoplaced)
+    (effects (font (size 1.27 1.27)) (justify right))
+    (property "Intersheetrefs" "${INTERSHEET_REFS}" (at 390.9603 249.0946 0)
+      (effects (font (size 1.27 1.27)) (justify right) hide)
+    )
