File: matrix_rgb.kicad_sch (KiCad schematic)
At the start: 217 parts, among them K1 ESC, K10 F9, K11 F10, K12 F11, K13 F12, K14 PRTSCR, K15 DELETE, K16 INSERT, K17 BACKTICK, K18 1, K19 2, K2 F1, K20 3, K21 4, K22 5, K23 6, K24 7, K25 8, K26 9, K27 0, K28 MINUS, K29 EQUAL, K3 F2, K30 BACKSPACE, K31 HOME, K32 TAB, K33 Q, K34 W, K35 E, K36 R, K37 T, K38 Y, K39 U, K4 F3, K40 I, K41 O, K42 P, K43 OBRAC, K44 CBRAC, K45 PAGEUP, K46 CAPS, K47 A, K48 S, K49 D, K5 F4, K50 F, K51 G, K52 H, K53 J, K54 K, K55 L, K56 SEMICOLON, K57 QUOTE, K58 HASH, K59 ISO ENTER, K6 F5, K60 PAGEDOWN, K61 LSHIFT, K62 BCKSLASH, K63 Z, K64 X, K65 C, K66 V, K67 B, K68 N, K69 M, K7 F6, K70 COMMA, K71 DOT, K72 SLASH, K73 RSHIFT, K74 UP, K75 END, K76 LCTRL, K77 LWIN, K78 LALT, K79 SPACE, K8 F7, K80 RALT(ALTGR), K81 FN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

Commit message: Schematic
Connections:
- net CS28: now also LED54.2 (BK); no longer LED54.3 (GK)
- net CS29: now also LED54.3 (GK); no longer LED54.4 (RK)
- net CS30: now also LED54.4 (RK); no longer LED54.2 (BK)
Changed lines of the file:
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@@
     )
   )
-  (global_label "CS29" (shape input) (at 298.704 328.676 180) (fields_autoplaced)
-    (effects (font (size 1.27 1.27)) (justify right))
-    (property "Intersheetrefs" "${INTERSHEET_REFS}" (at 291.3923 328.5966 0)
+  (global_label "CS29" (shape input) (at 298.704 333.756 180) (fields_autoplaced)
+    (effects (font (size 1.27 1.27)) (justify right))
+    (property "Intersheetrefs" "${INTERSHEET_REFS}" (at 291.3923 333.6766 0)
       (effects (font (size 1.27 1.27)) (justify right) hide)
     )
@@
     )
   )
-  (global_label "CS30" (shape input) (at 298.704 338.836 180) (fields_autoplaced)
-    (effects (font (size 1.27 1.27)) (justify right))
-    (property "Intersheetrefs" "${INTERSHEET_REFS}" (at 291.3923 338.7566 0)
+  (global_label "CS30" (shape input) (at 298.704 328.676 180) (fields_autoplaced)
+    (effects (font (size 1.27 1.27)) (justify right))
+    (property "Intersheetrefs" "${INTERSHEET_REFS}" (at 291.3923 328.5966 0)
       (effects (font (size 1.27 1.27)) (justify right) hide)
     )
@@
     )
   )
-  (global_label "CS28" (shape input) (at 298.704 333.756 180) (fields_autoplaced)
-    (effects (font (size 1.27 1.27)) (justify right))
-    (property "Intersheetrefs" "${INTERSHEET_REFS}" (at 291.3923 333.6766 0)
-      (effects (font (size 1.27 1.27)) (justify right) hide)
-    )
+  (global_label "CS28" (shape input) (at 298.704 338.836 180) (fields_autoplaced)
+    (effects (font (size 1.27 1.27)) (justify right))
+    (property "Intersheetrefs" "${INTERSHEET_REFS}" (at 291.3923 338.7566 0)
+      (effects (font (size 1.27 1.27)) (justify right) hide)
+    )

Commit message: PCB
Other:
- note removed: "ROW SPLIT"
Changed lines of the file:
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@@
     (effects (font (size 1.27 1.27)) (justify left bottom))
-  )
-  (text "ROW SPLIT" (at 295.148 209.55 0)
-    (effects (font (size 3 3)) (justify right bottom))
   )
   (text "LCTRL" (at 57.658 377.19 0)

Commit message: Schematic
Parts:
- S1, S2, S3: now left out of the parts list
Changed lines of the file:
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@@
   )
   (symbol (lib_id "marbastlib-mx:MX_stab") (at 508.508 122.174 0) (unit 1)
-    (in_bom yes) (on_board yes) (dnp no) (fields_autoplaced)
+    (in_bom no) (on_board yes) (dnp no) (fields_autoplaced)
     (property "Reference" "S1" (at 514.223 121.1385 0)
       (effects (font (size 1.27 1.27)) (justify left))
@@
   )
   (symbol (lib_id "marbastlib-mx:MX_stab") (at 508.508 129.032 0) (unit 1)
-    (in_bom yes) (on_board yes) (dnp no) (fields_autoplaced)
+    (in_bom no) (on_board yes) (dnp no) (fields_autoplaced)
     (property "Reference" "S2" (at 514.223 127.9965 0)
       (effects (font (size 1.27 1.27)) (justify left))
@@
   )
   (symbol (lib_id "marbastlib-mx:MX_stab") (at 508.508 136.906 0) (unit 1)
-    (in_bom yes) (on_board yes) (dnp no) (fields_autoplaced)
+    (in_bom no) (on_board yes) (dnp no) (fields_autoplaced)
     (property "Reference" "S3" (at 514.35 135.5089 0)
       (effects (font (size 1.27 1.27)) (justify left))

Commit message: Schematic
Parts:
- D10, D11, D12, D13, D14, D15, D16, D17, D18, D19, D2, D20, D21, D22, D23, D24, D25, D26, D27, D28, D29, D3, D30, D31, D32, D33, D34, D35, D36, D37, D38, D39, D4, D40, D41, D42, D43, D44, D45, D46, D47, D5, D6, D7, D8, D9: LCSC (none) -> C727123
- K1, K10, K11, K12, K13, K14, K15, K16, K17, K18, K19, K2, K20, K21, K22, K23, K24, K25, K26, K27, K28, K29, K3, K30, K31, K32, K33, K34, K35, K36, K37, K38, K39, K4, K40, K41, K42, K43, K44, K45, K46, K47, K48, K49, K5, K50, K51, K52, K53, K54, K55, K56, K57, K58, K59, K6, K60, K61, K62, K63, K64, K65, K66, K67, K68, K69, K7, K70, K71, K72, K73, K74, K75, K76, K77, K78, K79, K8, K80, K81, K82, K83, K84, K9: LCSC (none) -> C5184526
- LED1, LED10, LED11, LED12, LED13, LED14, LED15, LED16, LED17, LED18, LED19, LED2, LED20, LED21, LED22, LED23, LED24, LED25, LED26, LED27, LED28, LED29, LED3, LED30, LED31, LED32, LED33, LED34, LED35, LED36, LED37, LED38, LED39, LED4, LED40, LED41, LED42, LED43, LED44, LED45, LED46, LED47, LED48, LED49, LED5, LED50, LED51, LED52, LED53, LED54, LED55, LED56, LED57, LED58, LED59, LED6, LED60, LED61, LED62, LED63, LED64, LED65, LED66, LED67, LED68, LED69, LED7, LED70, LED71, LED72, LED73, LED74, LED75, LED76, LED77, LED78, LED79, LED8, LED80, LED81, LED82, LED83, LED84, LED9: LCSC (none) -> C409782
