File: ISO75+STM+PKRGB.kicad_sch (KiCad schematic)
At the start: 66 parts, among them J1 JST SH-4, Q1 2N7002, SW1 SW_Push, U1 XC6206P332MR, U2 STM32F072CBTx, U3 IS313741A

Commit message: Schematic
Parts:
- J1: value JST SH-4 -> Molex Pico
- R10, R13, R16, R19, R22, R25, R28, R31, R34, R37, R40: value 20Ω -> 51Ω
- R11, R14, R17, R20, R23, R26, R29, R32, R35, R38, R8: value 51Ω -> 20Ω
- U3: footprint acheron_Hardware:QFN-60-1EP_7x7mm_P0.4mm_EP5.4x5.4mm_ThermalReliefs -> PCM_marbastlib-various:QFN-60_EP_7x7_Pitch0.4mm
Other:
- moved on the sheet: C11, C12, C19, D1, R5, R6, R7, U1, U2

Commit message: PCB
Parts:
- J1: footprint Connector_JST:JST_SH_SM04B-SRSS-TB_1x04-1MP_P1.00mm_Horizontal -> Connector_Molex:Molex_Pico-EZmate_78171-0004_1x04-1MP_P1.20mm_Vertical
Changed lines of the file:
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@@
       (effects (font (size 1.27 1.27)) (justify left))
     )
-    (property "Footprint" "Connector_JST:JST_SH_SM04B-SRSS-TB_1x04-1MP_P1.00mm_Horizontal" (at 155.956 27.686 0)
+    (property "Footprint" "Connector_Molex:Molex_Pico-EZmate_78171-0004_1x04-1MP_P1.20mm_Vertical" (at 155.956 27.686 0)
       (effects (font (size 1.27 1.27)) hide)
     )

Commit message: PCB
Parts:
- R5, R6: value 4.7kΩ -> 2kΩ
Other:
- note added: "Aproximately 14.07mA per channel."
- note added: "LED DRIVER"
- note added: "MICROCONTROLLER"
Changed lines of the file:
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@@
+    (effects (font (size 1.27 1.27)) (justify left bottom))
+  )
+  (text "LED DRIVER" (at 105.5624 59.2836 0)
     (effects (font (size 1.27 1.27)) (justify left bottom))
   )
@@
     (effects (font (size 1.27 1.27)) (justify left bottom))
   )
+  (text "MICROCONTROLLER" (at 83.7184 59.4868 0)
+    (effects (font (size 1.27 1.27)) (justify left bottom))
+  )
   (text "14/11/2022" (at 206.502 194.31 0)
     (effects (font (size 1.27 1.27)) (justify left bottom))
@@
   )
   (text "VOLTAGE SHIFTER" (at 38.354 51.308 0)
+    (effects (font (size 1.27 1.27)) (justify left bottom))
+  )
+  (text "Aproximately 14.07mA per channel." (at 105.5116 61.8744 0)
     (effects (font (size 1.27 1.27)) (justify left bottom))
   )
@@
       (effects (font (size 1.27 1.27)) (justify left))
     )
-    (property "Value" "4.7kΩ" (at 35.814 117.221 0)
+    (property "Value" "2kΩ" (at 35.814 117.221 0)
       (effects (font (size 1.27 1.27)) (justify left))
     )
@@
       (effects (font (size 1.27 1.27)) (justify left))
     )
-    (property "Value" "4.7kΩ" (at 22.606 116.967 0)
-      (effects (font (size 1.27 1.27)) (justify left))
-    )
+    (property "Value" "2kΩ" (at 22.606 116.967 0)
+      (effects (font (size 1.27 1.27)) (justify left))
+    )

Commit message: Schematic
Parts:
- C15: value 1uf -> 1uF
- J1: LCSC (none) -> C588524
- R10, R13, R16, R19, R22, R25, R28, R31, R34, R37, R40: LCSC C25741 -> C25125
- R11, R12, R14, R15, R17, R18, R20, R21, R23, R24, R26, R27, R29, R30, R32, R33, R35, R36, R38, R39, R8, R9: LCSC C25741 -> C25150
- R4: LCSC C25551 -> C138022
- SW1: LCSC (none) -> C92584
- U1: LCSC (none) -> C5446
- U3: LCSC C2940604 -> C2844697
Changed lines of the file:
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@@
+      (effects (font (size 1.27 1.27)) hide)
+    )
+    (property "LCSC" "C92584" (at 176.276 27.178 0)
       (effects (font (size 1.27 1.27)) hide)
     )
@@
       (effects (font (size 1.27 1.27)) hide)
     )
-    (property "LCSC" "C25741" (at 155.448 95.758 0)
+    (property "LCSC" "C25150" (at 155.448 95.758 0)
       (effects (font (size 1.27 1.27)) hide)
     )
@@
       (effects (font (size 1.27 1.27)) hide)
     )
-    (property "LCSC" "C25741" (at 155.448 110.998 0)
+    (property "LCSC" "C25150" (at 155.448 110.998 0)
       (effects (font (size 1.27 1.27)) hide)
     )
@@
       (effects (font (size 1.27 1.27)) hide)
     )
-    (property "LCSC" "C25741" (at 155.448 154.178 0)
+    (property "LCSC" "C25125" (at 155.448 154.178 0)
       (effects (font (size 1.27 1.27)) hide)
     )
@@
       (effects (font (size 1.27 1.27)) hide)
     )
-    (property "LCSC" "C25741" (at 155.448 149.098 0)
+    (property "LCSC" "C25150" (at 155.448 149.098 0)
       (effects (font (size 1.27 1.27)) hide)
     )
@@
       (effects (font (size 1.27 1.27)) hide)
     )
-    (property "LCSC" "C25741" (at 155.448 121.158 0)
+    (property "LCSC" "C25150" (at 155.448 121.158 0)
       (effects (font (size 1.27 1.27)) hide)
     )
@@
       (effects (font (size 1.27 1.27)) hide)
     )
-    (property "LCSC" "C25741" (at 155.448 161.798 0)
+    (property "LCSC" "C25125" (at 155.448 161.798 0)
       (effects (font (size 1.27 1.27)) hide)
     )
@@
     )
     (property "Datasheet" "~" (at 155.956 27.686 0)
+      (effects (font (size 1.27 1.27)) hide)
+    )
+    (property "LCSC" "C588524" (at 155.956 27.686 0)
       (effects (font (size 1.27 1.27)) hide)
     )
@@
       (effects (font (size 1.27 1.27)) hide)
     )
-    (property "LCSC" "C25741" (at 155.448 128.778 0)
+    (property "LCSC" "C25150" (at 155.448 128.778 0)
       (effects (font (size 1.27 1.27)) hide)
     )
@@
       (effects (font (size 1.27 1.27)) hide)
     )
-    (property "LCSC" "C25741" (at 155.448 105.918 0)
+    (property "LCSC" "C25150" (at 155.448 105.918 0)
       (effects (font (size 1.27 1.27)) hide)
     )
@@
       (effects (font (size 1.27 1.27)) hide)
     )
-    (property "LCSC" "C25741" (at 155.448 118.618 0)
+    (property "LCSC" "C25150" (at 155.448 118.618 0)
       (effects (font (size 1.27 1.27)) hide)
     )
@@
       (effects (font (size 1.27 1.27)) hide)
     )
-    (property "LCSC" "C25741" (at 155.448 133.858 0)
+    (property "LCSC" "C25150" (at 155.448 133.858 0)
       (effects (font (size 1.27 1.27)) hide)
     )
@@
       (effects (font (size 1.27 1.27)) (justify left))
     )
-    (property "Value" "1uf" (at 238.252 67.3162 0)
+    (property "Value" "1uF" (at 238.252 67.3162 0)
       (effects (font (size 1.27 1.27)) (justify left))
     )
@@
       (effects (font (size 1.27 1.27)) hide)
     )
-    (property "LCSC" "C25741" (at 155.448 138.938 0)
+    (property "LCSC" "C25125" (at 155.448 138.938 0)
       (effects (font (size 1.27 1.27)) hide)
     )
@@
       (effects (font (size 1.27 1.27)) hide)
     )
-    (property "LCSC" "C25741" (at 155.448 98.298 0)
+    (property "LCSC" "C25150" (at 155.448 98.298 0)
       (effects (font (size 1.27 1.27)) hide)
     )
@@
       (effects (font (size 1.27 1.27)) hide)
     )
+    (property "LCSC" "C5446" (at 33.02 34.29 0)
+      (effects (font (size 1.27 1.27)) hide)
+    )
     (pin "1")
     (pin "2")
@@
       (effects (font (size 1.27 1.27)) hide)
     )
-    (property "LCSC" "C25741" (at 155.448 131.318 0)
+    (property "LCSC" "C25125" (at 155.448 131.318 0)
       (effects (font (size 1.27 1.27)) hide)
     )
@@
       (effects (font (size 1.27 1.27)) hide)
     )
-    (property "LCSC" "C25741" (at 155.448 80.518 0)
+    (property "LCSC" "C25150" (at 155.448 80.518 0)
       (effects (font (size 1.27 1.27)) hide)
     )
@@
       (effects (font (size 1.27 1.27)) hide)
     )
-    (property "LCSC" "C25741" (at 155.448 88.138 0)
+    (property "LCSC" "C25150" (at 155.448 88.138 0)
       (effects (font (size 1.27 1.27)) hide)
     )
@@
       (effects (font (size 1.27 1.27)) hide)
     )
-    (property "LCSC" "C2940604" (at 137.668 128.778 0)
+    (property "LCSC" "C2844697" (at 137.668 128.778 0)
       (effects (font (size 1.27 1.27)) hide)
     )
@@
       (effects (font (size 1.27 1.27)) hide)
     )
-    (property "LCSC" "C25741" (at 155.448 151.638 0)
+    (property "LCSC" "C25150" (at 155.448 151.638 0)
       (effects (font (size 1.27 1.27)) hide)
     )
@@
       (effects (font (size 1.27 1.27)) hide)
     )
-    (property "LCSC" "C25551" (at 114.808 98.298 0)
+    (property "LCSC" "C138022" (at 114.808 98.298 0)
       (effects (font (size 1.27 1.27)) hide)
     )
@@
       (effects (font (size 1.27 1.27)) hide)
     )
-    (property "LCSC" "C25741" (at 155.448 90.678 0)
+    (property "LCSC" "C25150" (at 155.448 90.678 0)
       (effects (font (size 1.27 1.27)) hide)
     )
@@
       (effects (font (size 1.27 1.27)) hide)
     )
-    (property "LCSC" "C25741" (at 155.448 85.598 0)
+    (property "LCSC" "C25125" (at 155.448 85.598 0)
       (effects (font (size 1.27 1.27)) hide)
     )
@@
       (effects (font (size 1.27 1.27)) hide)
     )
-    (property "LCSC" "C25741" (at 155.448 136.398 0)
+    (property "LCSC" "C25150" (at 155.448 136.398 0)
       (effects (font (size 1.27 1.27)) hide)
     )
@@
       (effects (font (size 1.27 1.27)) hide)
     )
-    (property "LCSC" "C25741" (at 155.448 100.838 0)
+    (property "LCSC" "C25125" (at 155.448 100.838 0)
       (effects (font (size 1.27 1.27)) hide)
     )
@@
       (effects (font (size 1.27 1.27)) hide)
     )
-    (property "LCSC" "C25741" (at 155.448 103.378 0)
+    (property "LCSC" "C25150" (at 155.448 103.378 0)
       (effects (font (size 1.27 1.27)) hide)
     )
@@
       (effects (font (size 1.27 1.27)) hide)
     )
-    (property "LCSC" "C25741" (at 155.448 113.538 0)
+    (property "LCSC" "C25150" (at 155.448 113.538 0)
       (effects (font (size 1.27 1.27)) hide)
     )
@@
       (effects (font (size 1.27 1.27)) hide)
     )
-    (property "LCSC" "C25741" (at 155.448 93.218 0)
+    (property "LCSC" "C25125" (at 155.448 93.218 0)
       (effects (font (size 1.27 1.27)) hide)
     )
@@
       (effects (font (size 1.27 1.27)) hide)
     )
-    (property "LCSC" "C25741" (at 155.448 156.718 0)
+    (property "LCSC" "C25150" (at 155.448 156.718 0)
       (effects (font (size 1.27 1.27)) hide)
     )
@@
       (effects (font (size 1.27 1.27)) hide)
     )
-    (property "LCSC" "C25741" (at 155.448 108.458 0)
+    (property "LCSC" "C25125" (at 155.448 108.458 0)
       (effects (font (size 1.27 1.27)) hide)
     )
@@
       (effects (font (size 1.27 1.27)) hide)
     )
-    (property "LCSC" "C25741" (at 155.448 83.058 0)
+    (property "LCSC" "C25150" (at 155.448 83.058 0)
       (effects (font (size 1.27 1.27)) hide)
     )
@@
       (effects (font (size 1.27 1.27)) hide)
     )
-    (property "LCSC" "C25741" (at 155.448 123.698 0)
+    (property "LCSC" "C25125" (at 155.448 123.698 0)
       (effects (font (size 1.27 1.27)) hide)
     )
@@
       (effects (font (size 1.27 1.27)) hide)
     )
-    (property "LCSC" "C25741" (at 155.448 144.018 0)
+    (property "LCSC" "C25150" (at 155.448 144.018 0)
       (effects (font (size 1.27 1.27)) hide)
     )
@@
       (effects (font (size 1.27 1.27)) hide)
     )
-    (property "LCSC" "C25741" (at 155.448 141.478 0)
+    (property "LCSC" "C25150" (at 155.448 141.478 0)
       (effects (font (size 1.27 1.27)) hide)
     )
@@
       (effects (font (size 1.27 1.27)) hide)
     )
-    (property "LCSC" "C25741" (at 155.448 126.238 0)
+    (property "LCSC" "C25150" (at 155.448 126.238 0)
       (effects (font (size 1.27 1.27)) hide)
     )
@@
       (effects (font (size 1.27 1.27)) hide)
     )
-    (property "LCSC" "C25741" (at 155.448 116.078 0)
+    (property "LCSC" "C25125" (at 155.448 116.078 0)
       (effects (font (size 1.27 1.27)) hide)
     )
@@
       (effects (font (size 1.27 1.27)) hide)
     )
-    (property "LCSC" "C25741" (at 155.448 146.558 0)
+    (property "LCSC" "C25125" (at 155.448 146.558 0)
       (effects (font (size 1.27 1.27)) hide)
     )
@@
       (effects (font (size 1.27 1.27)) hide)
     )
-    (property "LCSC" "C25741" (at 155.448 159.258 0)
-      (effects (font (size 1.27 1.27)) hide)
-    )
+    (property "LCSC" "C25150" (at 155.448 159.258 0)
+      (effects (font (size 1.27 1.27)) hide)
+    )
